Commit message: Add files via upload

File: urdf/aprs_lab_robots.urdf.xacro (robot description, xacro)
@@ -2,10 +2,33 @@
 <robot xmlns:xacro="http://www.ros.org/wiki/xacro" name="aprs_lab_robots">
   <link name="world"/>
+  <link name="aprs_ur_base_link"/>
+  <link name="aprs_fanuc_base_link"/>
+  <joint name = "ur_world_to_base" type = "fixed">
+    <origin rpy = "0 0 0" xyz = "10 0 0"/>
+    <parent link = "world"/>
+    <child link = "aprs_ur_base_link"/>
+  </joint>
+  <joint name = "fanuc_world_to_base" type = "fixed">
+    <origin rpy = "0 0 0" xyz = "0 10 0"/>
+    <parent link = "world"/>
+    <child link = "aprs_fanuc_base_link"/>
+  </joint>
+  <joint name = "franka_world_to_base" type = "fixed">
+    <origin rpy = "0 0 0" xyz = "0 0 0"/>
+    <parent link = "world"/>
+    <child link = "aprs_franka_base_link"/>
+  </joint>
   <xacro:include filename="$(find aprs_description)/urdf/ur/aprs_ur_macro.xacro"/>
+  <xacro:include filename="$(find aprs_description)/urdf/fanuc/aprs_fanuc_macro.xacro"/>
+  <xacro:include filename="$(find aprs_description)/urdf/franka/aprs_franka_macro.xacro"/>
     <!-- ROS2 Control Plugin -->
   <xacro:arg name="controllers" default="$(find aprs_description)/config/robot_controllers.yaml" />
   <xacro:aprs_ur
-    parent="world">
+    parent="aprs_ur_base_link">
   </xacro:aprs_ur>
+  <xacro:aprs_fanuc
+    parent="aprs_fanuc_base_link">
+  </xacro:aprs_fanuc>
+  <xacro:aprs_franka></xacro:aprs_franka>
   <gazebo>
     <plugin filename="libgz_ros2_control-system.so" name="gz_ros2_control::GazeboSimROS2ControlPlugin">
